Commit message: joystic works with gazebo model

File: src/panporter_pkg/urdf/panporter.urdf.xacro (robot description, xacro)
@@ -4,4 +4,5 @@
   <link name="base_footprint"/>
   <joint name="base_joint" type="fixed">
+    <pose>0 0 0.36 0 0 0</pose>
     <parent link="base_footprint"/>
     <child link="robot_cover" />
@@ -12,24 +13,25 @@
     <visual>
       <geometry>
-        <mesh filename="package://panporter_pkg/urdf/robot_cover.stl" scale="1.0 1.0 1.0"/>
-      </geometry>
-      <origin rpy="0 0 -1.570796327" xyz="0 0 0"/>
-      <!-- <material name="yellow">
+        <mesh filename="package://panporter_pkg/meshes/robot_parts/robot_cover.stl" scale="1.0 1.0 1.0"/>
+      </geometry>
+      <origin rpy="0 0 0" xyz="0 0 0"/>
+      <material name="yellow">
         <color rgba="1 1 0 0.4"/>
-      </material> -->
-    </visual>
-    <collision>
-      <geometry>
-        <mesh filename="package://panporter_pkg/urdf/robot_cover.stl" scale="1.0 1.0 1.0"/>
-      </geometry>
-      <origin rpy="0 0 -1.570796327" xyz="0 0 0"/>
-      <!-- <material name="yellow">
+      </material>
+    </visual>
+    <collision>
+      <origin rpy="0 0 0" xyz="0 0 0"/>
+      <geometry>
+        <mesh filename="package://panporter_pkg/meshes/robot_parts/robot_cover.stl" scale="1.0 1.0 1.0"/>
+      </geometry>
+      <material name="yellow">
         <color rgba="1 1 0 0.4"/>
-      </material> -->
+      </material>
     </collision>
     <inertial>
 	    <mass value="10.0"/>
-	    <inertia ixx="1.0" ixy="0.1" ixz="0.1" iyy="1.0" iyz="0.1" izz="1.0"/>
-      <origin rpy="0 0 -1.570796327" xyz="0 0 0"/>
+  <!-- izz=skrecanie, iyy=obracanie_bebnem, ixx=pochylanie_na_boki -->
+	    <inertia ixx="0.358333333" ixy="0.0" ixz="0.0" iyy="0.358333333" iyz="0.0" izz="0.450"/>
+      <origin rpy="0 0 0" xyz="0 0 -0.1"/>
     </inertial>
   </link>
@@ -40,43 +42,5 @@
     <mu2> 10.0 </mu2>
   </gazebo> -->
-  <joint name="prism_left_joint" type="prismatic">
-    <parent link="robot_cover"/>
-    <child link="prism_left_blue_link"/>
-    <origin rpy="0 0 0" xyz="0 0.2 0"/>
-    <axis xyz="1 0 0" />
-    <limit effort="300" velocity="1.0" lower="-0.1" upper="0.1"/>
-    <safety_controller k_position="20" k_velocity="20" soft_lower_limit="-0.15" soft_upper_limit="0.15"/>
-    <dynamics damping="50" friction="1.0"/>
-  </joint>
-  <joint name="prism_right_joint" type="prismatic">
-    <parent link="robot_cover"/>
-    <child link="prism_right_blue_link"/>
-    <origin rpy="0 0 0" xyz="0 -0.2 0"/>
-    <axis xyz="1 0 0" />
-    <limit effort="300" velocity="1.0" lower="-0.1" upper="0.1"/>
-    <safety_controller k_position="20" k_velocity="20" soft_lower_limit="-0.15" soft_upper_limit="0.15"/>
-    <dynamics damping="50" friction="1.0"/>
-  </joint>
-  <transmission name="prism_left_trans">
-    <type>transmission_interface/SimpleTransmission</type>
-    <joint name="prism_left_joint">
-      <hardwareInterface>hardware_interface/EffortJointInterface</hardwareInterface>
-    </joint>
-    <actuator name="prism_left_motor">
-      <mechanicalReduction>1</mechanicalReduction>
-      <hardwareInterface>hardware_interface/EffortJointInterface</hardwareInterface>
-    </actuator>
-  </transmission>
-  <transmission name="prism_right_trans">
-    <type>transmission_interface/SimpleTransmission</type>
-    <joint name="prism_right_joint">
-      <hardwareInterface>hardware_interface/EffortJointInterface</hardwareInterface>
-    </joint>
-    <actuator name="prism_right_motor">
-      <mechanicalReduction>1</mechanicalReduction>
-      <hardwareInterface>hardware_interface/EffortJointInterface</hardwareInterface>
-    </actuator>
-  </transmission>
-  <link name="prism_left_blue_link">
+  <link name="prism_left_link">
     <pose>0 0 0.35 0 0 0</pose>
     <visual>
@@ -96,9 +60,9 @@
     </collision>
     <inertial>
-	    <mass value="0.1"/>
-	    <inertia ixx="0.01" ixy="0.1" ixz="0.1" iyy="0.01" iyz="0.1" izz="0.01"/>
-    </inertial>
-  </link>
-  <link name="prism_right_blue_link">
+	    <mass value="0.5"/>
+	    <inertia ixx="0.001716667" ixy="0.0" ixz="0.0" iyy="0.001716667" iyz="0.0" izz="0.1"/>
+    </inertial>
+  </link>
+  <link name="prism_right_link">
     <pose>0 0 0.35 0 0 0</pose>
     <visual>
@@ -118,23 +82,29 @@
     </collision>
     <inertial>
-	    <mass value="0.1"/>
-	    <inertia ixx="0.01" ixy="0.1" ixz="0.1" iyy="0.01" iyz="0.1" izz="0.01"/>
-    </inertial>
-  </link>
-  <joint name="wheel_left_joint" type="continuous">
-    <parent link="prism_left_blue_link"/>
-    <child link="wheel_left_link"/>
-    <origin rpy="0 0 0" xyz="0 0.1 0"/>
-    <axis xyz="0 1 0" />
-    <limit effort="300" velocity="10000"/>
-    <dynamics damping="50" friction="1"/>
-  </joint>
-  <transmission name="wheel_left_trans">
+	    <mass value="0.5"/>
+	    <inertia ixx="0.001716667" ixy="0.0" ixz="0.0" iyy="0.001716667" iyz="0.0" izz="0.1"/>
+    </inertial>
+  </link>
+  <joint name="prism_right_blue_joint" type="fixed">
+    <parent link="prism_left_link"/>
+    <child link="prism_right_link"/>
+    <origin xyz="0 -0.4 0"/>
+  </joint>
+  <joint name="prism_joint" type="prismatic">
+    <parent link="robot_cover"/>
+    <child link="prism_left_link"/>
+    <origin rpy="0 0 0" xyz="0 0.2 0"/>
+    <axis xyz="1 0 0" />
+    <limit effort="3000" velocity="10.0" lower="-0.5" upper="0.5"/>
+    <safety_controller k_position="20" k_velocity="20" soft_lower_limit="-0.45" soft_upper_limit="0.45"/>
+    <dynamics damping="5" friction="1.0"/>
+  </joint>
+  <transmission name="prism_trans">
     <type>transmission_interface/SimpleTransmission</type>
-    <joint name="wheel_left_joint">
+    <joint name="prism_joint">
       <hardwareInterface>hardware_interface/EffortJointInterface</hardwareInterface>
     </joint>
-    <actuator name="wheel_left_motor">
-      <mechanicalReduction>10</mechanicalReduction>
+    <actuator name="prism_motor">
+      <mechanicalReduction>1</mechanicalReduction>
       <hardwareInterface>hardware_interface/EffortJointInterface</hardwareInterface>
     </actuator>
@@ -144,7 +114,7 @@
     <visual>
       <geometry>
-        <mesh filename="package://panporter_pkg/urdf/wheel.stl" scale="1.0 1.0 1.0"/>
-      </geometry>
-      <origin rpy="1.570796327 0 0" xyz="0 0 0"/>
+        <mesh filename="package://panporter_pkg/meshes/robot_parts/wheel.stl" scale="1.0 1.0 1.0"/>
+      </geometry>
+      <origin rpy="0 0 0" xyz="0 0 0"/>
       <!-- <material name="red">
         <color rgba="1 0 0 0.4"/>
@@ -152,31 +122,29 @@
     </visual>
     <collision>
-      <geometry>
-        <mesh filename="package://panporter_pkg/urdf/wheel.stl" scale="1.0 1.0 1.0"/>
-      </geometry>
-      <origin rpy="1.570796327 0 0" xyz="0 0 0"/>
+      <origin rpy="0 0 0" xyz="0 0 0"/>
+      <geometry>
+        <mesh filename="package://panporter_pkg/meshes/robot_parts/wheel.stl" scale="1.0 1.0 1.0"/>
+      </geometry>
+      <surface></surface>
     </collision>
     <inertial>
 	    <mass value="1"/>
-	    <inertia ixx="0.5" ixy="0.1" ixz="0.1" iyy="0.5" iyz="0.1" izz="0.5"/>
-    </inertial>
-  </link>
-  <!-- <gazebo reference="wheel_left_link">
-    <material>Gazebo/Green</material>
-  </gazebo> -->
-  <joint name="wheel_right_joint" type="continuous">
-    <parent link="prism_right_blue_link"/>
-    <child link="wheel_right_link"/>
-    <origin rpy="0 0 0" xyz="0 -0.1 0"/>
+	    <inertia ixx="0.07945" ixy="0.0" ixz="0.01" iyy="0.1389" iyz="0.0" izz="0.07945"/>
+    </inertial>
+  </link>
+  <joint name="wheel_left_joint" type="continuous">
+    <parent link="prism_left_link"/>
+    <child link="wheel_left_link"/>
+    <origin rpy="0 0 0" xyz="0 0.1 0"/>
     <axis xyz="0 1 0" />
-    <limit effort="300" velocity="10000"/> <!-- lower="-1.570796327" upper="1.570796327"/> -->
-    <dynamics damping="50" friction="1"/>
-  </joint>
-  <transmission name="wheel_right_trans">
+    <limit effort="50" velocity="10000"/>
+    <dynamics damping="5" friction="1"/>
+  </joint>
+  <transmission name="wheel_left_trans">
     <type>transmission_interface/SimpleTransmission</type>
-    <joint name="wheel_right_joint">
+    <joint name="wheel_left_joint">
       <hardwareInterface>hardware_interface/EffortJointInterface</hardwareInterface>
     </joint>
-    <actuator name="wheel_right_motor">
+    <actuator name="wheel_left_motor">
       <mechanicalReduction>10</mechanicalReduction>
       <hardwareInterface>hardware_interface/EffortJointInterface</hardwareInterface>
@@ -187,7 +155,7 @@
     <visual>
       <geometry>
-        <mesh filename="package://panporter_pkg/urdf/wheel.stl" scale="1.0 1.0 1.0"/>
-      </geometry>
-      <origin rpy="1.570796327 0 0" xyz="0 0 0"/>
+        <mesh filename="package://panporter_pkg/meshes/robot_parts/wheel.stl" scale="1.0 1.0 1.0"/>
+      </geometry>
+      <origin rpy="0 0 0" xyz="0 0 0"/>
       <!-- <material name="red">
         <color rgba="1 0 0 0.4"/>
@@ -196,16 +164,31 @@
     <collision>
       <geometry>
-        <mesh filename="package://panporter_pkg/urdf/wheel.stl" scale="1.0 1.0 1.0"/>
-      </geometry>
-      <origin rpy="1.570796327 0 0" xyz="0 0 0"/>
+        <mesh filename="package://panporter_pkg/meshes/robot_parts/wheel.stl" scale="1.0 1.0 1.0"/>
+      </geometry>
+      <origin rpy="0 0 0" xyz="0 0 0"/>
     </collision>
     <inertial>
 	    <mass value="1"/>
-	    <inertia ixx="0.5" ixy="0.1" ixz="0.1" iyy="0.5" iyz="0.1" izz="0.5"/>
-    </inertial>
-  </link>
-  <!-- <gazebo reference="wheel_left_link">
-    <material>Gazebo/Red</material>
-  </gazebo> -->
+	    <inertia ixx="0.07945" ixy="0.0" ixz="0.01" iyy="0.1389" iyz="0.0" izz="0.07945"/>
+    </inertial>
+  </link>
+  <joint name="wheel_right_joint" type="continuous">
+    <parent link="prism_right_link"/>
+    <child link="wheel_right_link"/>
+    <origin rpy="0 0 0" xyz="0 -0.1 0"/>
+    <axis xyz="0 1 0" />
+    <limit effort="50" velocity="10000"/> <!-- lower="-1.570796327" upper="1.570796327"/> -->
+    <dynamics damping="5" friction="1"/>
+  </joint>
+  <transmission name="wheel_right_trans">
+    <type>transmission_interface/SimpleTransmission</type>
+    <joint name="wheel_right_joint">
+      <hardwareInterface>hardware_interface/EffortJointInterface</hardwareInterface>
+    </joint>
+    <actuator name="wheel_right_motor">
+      <mechanicalReduction>10</mechanicalReduction>
+      <hardwareInterface>hardware_interface/EffortJointInterface</hardwareInterface>
+    </actuator>
+  </transmission>
   <joint name="imu_joint" type="fixed">
     <parent link="robot_cover"/>
@@ -223,5 +206,5 @@
       <origin xyz="0 0 0" rpy="0 0 0"/>
       <geometry>
-        <mesh filename="package://turtlebot3_description/meshes/sensors/lds.stl" scale="0.001 0.001 0.001"/>
+        <mesh filename="package://panporter_pkg/meshes/sensors/lds.stl" scale="0.001 0.001 0.001"/>
       </geometry>
       <material name="dark"/>
@@ -236,11 +219,11 @@
       <mass value="0.114" />
       <origin xyz="0 0 0" />
-      <inertia ixx="0.001" ixy="0.1" ixz="0.1"
-               iyy="0.001" iyz="0.1"
+      <inertia ixx="0.001" ixy="0.0" ixz="0.0"
+               iyy="0.001" iyz="0.0"
                izz="0.001" />
     </inertial>
   </link>
   <joint name="camera_joint" type="fixed">
-    <origin xyz="0.064 -0.065 0.094" rpy="0 0 0"/>
+    <origin xyz="0.2 0 0.2" rpy="0 0 0"/>
     <parent link="robot_cover"/>
     <child link="camera_link"/>
@@ -248,12 +231,12 @@
   <link name="camera_link">
     <visual>
-      <origin xyz="0.003 2.065 0.007" rpy="0 0 0"/>
+      <origin xyz="0 0 0" rpy="1.570796327 0 1.570796327"/>
       <geometry>
        <!-- <mesh filename="package://turtlebot3_gazebo/models/kinect/meshes/kinect.dae" /> -->
-       <mesh filename="package://turtlebot3_description/meshes/sensors/lds.stl"  scale="0.001 0.001 0.001"/>
-      </geometry>
-    </visual>
-    <collision>
-      <origin xyz="0.003 2.065 0.007" rpy="0 0 0"/>
+       <mesh filename="package://panporter_pkg/meshes/sensors/zed2.dae"/>
+      </geometry>
+    </visual>
+    <collision>
+      <origin xyz="0 0 0" rpy="0 0 1.570796327"/>
       <geometry>
         <box size="0.012 0.132 0.020"/>
@@ -261,11 +244,11 @@
     </collision>
     <!-- This inertial field needs doesn't contain reliable data!! -->
-    <inertial>
+<!--   <inertial>
       <mass value="0.564" />
       <origin xyz="0 0 0" />
-      <inertia ixx="0.003881243" ixy="0.1" ixz="0.1"
-               iyy="0.000498940" iyz="0.1"
+      <inertia ixx="0.003881243" ixy="0.0" ixz="0.0"
+               iyy="0.000498940" iyz="0.0"
                izz="0.003879257" />
-    </inertial>
+    </inertial>-->
   </link>
   <gazebo>
@@ -297,5 +280,5 @@
       <robotNamespace>/panporter</robotNamespace>
       <robotSimType>gazebo_ros_control/DefaultRobotHWSim</robotSimType>
-      <controlPeriod>0.002</controlPeriod>
+      <controlPeriod>0.001</controlPeriod>
       <legacyModeNS>false</legacyModeNS>
     </plugin>
@@ -313,12 +296,14 @@
   <!-- robot_cover -->
 	<gazebo reference="robot_cover">
-		<material value="Gazebo/Grey"/>
+		<material value="Gazebo/Yellow"/>
+    <mu1>100.0</mu1>
+    <mu2>100.0</mu2>
 	</gazebo>
-  <!-- prism_left_blue_link -->
-	<gazebo reference="prism_left_blue_link">
+  <!-- prism_left_link -->
+	<gazebo reference="prism_left_link">
 		<material value="Gazebo/Blue"/>
 	</gazebo>
-  <!-- prism_right_blue_link -->
-	<gazebo reference="prism_right_blue_link">
+  <!-- prism_right_link -->
+	<gazebo reference="prism_right_link">
 		<material value="Gazebo/Blue"/>
 	</gazebo>
@@ -326,8 +311,12 @@
 	<gazebo reference="wheel_left_link">
 		<material value="Gazebo/Red"/>
+    <mu1>100.0</mu1>
+    <mu2>100.0</mu2>
 	</gazebo>
   <!-- wheel_right_link -->
 	<gazebo reference="wheel_right_link">
-		<material value="Gazebo/Red"/>
+		<material value="Gazebo/Green"/>
+    <mu1>100.0</mu1>
+    <mu2>100.0</mu2>
 	</gazebo>
   <gazebo>

Commit message: added pid controller

File: src/panporter_pkg/urdf/panporter.urdf.xacro (robot description, xacro)
@@ -95,9 +95,32 @@
     <child link="prism_left_link"/>
     <origin rpy="0 0 0" xyz="0 0.2 0"/>
-    <axis xyz="1 0 0" />
+    <axis xyz="-1 0 0" />
     <limit effort="3000" velocity="10.0" lower="-0.5" upper="0.5"/>
     <safety_controller k_position="20" k_velocity="20" soft_lower_limit="-0.45" soft_upper_limit="0.45"/>
     <dynamics damping="5" friction="1.0"/>
   </joint>
+  <!-- <joint name="spring_joint" type="prismatic">
+    <parent link="base_link"/>
+    <child link="prism_right_link"/>
+    <origin xyz="0 -0.2 0"/>
+    <axis>
+      <xyz>1 0 0</xyz>
+      <limit lower="-0.001" upper="0.001"/>
+      <safety_controller k_position="20" k_velocity="20" soft_lower_limit="-0.15" soft_upper_limit="0.15"/>
+      <dynamics spring_stiffness="250" spring_reference="0.06" damping="50" friction="0.75"/>
+      <use_parent_model_frame>0</use_parent_model_frame>
+      <dynamics damping="50" friction="1.0"/>
+    <axis/>
+    <physics>
+      <ode>
+        <implicit_spring_damper>1</implicit_spring_damper>
+        <cfm_damping>1</cfm_damping>
+        <limit>
+          <cfm>0</cfm>
+          <erp>0.2</erp>
+        </limit>
+      </ode>
+    </physics>
+  </joint> -->
   <transmission name="prism_trans">
     <type>transmission_interface/SimpleTransmission</type>

Commit message: second pid controller for linear component of wheels velocity

File: src/panporter_pkg/urdf/panporter.urdf.xacro (robot description, xacro)
@@ -96,7 +96,7 @@
     <origin rpy="0 0 0" xyz="0 0.2 0"/>
     <axis xyz="-1 0 0" />
-    <limit effort="3000" velocity="10.0" lower="-0.5" upper="0.5"/>
+    <limit effort="3000" velocity="50.0" lower="-0.5" upper="0.5"/>
     <safety_controller k_position="20" k_velocity="20" soft_lower_limit="-0.45" soft_upper_limit="0.45"/>
-    <dynamics damping="5" friction="1.0"/>
+    <dynamics damping="0.01" friction="0.1"/>
   </joint>
   <!-- <joint name="spring_joint" type="prismatic">
@@ -108,7 +108,7 @@
       <limit lower="-0.001" upper="0.001"/>
       <safety_controller k_position="20" k_velocity="20" soft_lower_limit="-0.15" soft_upper_limit="0.15"/>
-      <dynamics spring_stiffness="250" spring_reference="0.06" damping="50" friction="0.75"/>
+      <dynamics spring_stiffness="250" spring_reference="0.06" damping="0.1" friction="0.75"/>
       <use_parent_model_frame>0</use_parent_model_frame>
-      <dynamics damping="50" friction="1.0"/>
+      <dynamics damping="0.1" friction="1.0"/>
     <axis/>
     <physics>
@@ -137,5 +137,5 @@
     <visual>
       <geometry>
-        <mesh filename="package://panporter_pkg/meshes/robot_parts/wheel.stl" scale="1.0 1.0 1.0"/>
+        <mesh filename="package://panporter_pkg/meshes/robot_parts/wheel2.stl" scale="0.001 0.001 0.001"/>
       </geometry>
       <origin rpy="0 0 0" xyz="0 0 0"/>
@@ -147,5 +147,5 @@
       <origin rpy="0 0 0" xyz="0 0 0"/>
       <geometry>
-        <mesh filename="package://panporter_pkg/meshes/robot_parts/wheel.stl" scale="1.0 1.0 1.0"/>
+        <mesh filename="package://panporter_pkg/meshes/robot_parts/wheel2.stl" scale="0.001 0.001 0.001"/>
       </geometry>
       <surface></surface>
@@ -161,6 +161,6 @@
     <origin rpy="0 0 0" xyz="0 0.1 0"/>
     <axis xyz="0 1 0" />
-    <limit effort="50" velocity="10000"/>
-    <dynamics damping="5" friction="1"/>
+    <limit effort="500" velocity="1000"/>
+    <dynamics damping="0.1" friction="0.1"/>
   </joint>
   <transmission name="wheel_left_trans">
@@ -178,5 +178,5 @@
     <visual>
       <geometry>
-        <mesh filename="package://panporter_pkg/meshes/robot_parts/wheel.stl" scale="1.0 1.0 1.0"/>
+        <mesh filename="package://panporter_pkg/meshes/robot_parts/wheel2.stl" scale="0.001 0.001 0.001"/>
       </geometry>
       <origin rpy="0 0 0" xyz="0 0 0"/>
@@ -187,5 +187,5 @@
     <collision>
       <geometry>
-        <mesh filename="package://panporter_pkg/meshes/robot_parts/wheel.stl" scale="1.0 1.0 1.0"/>
+        <mesh filename="package://panporter_pkg/meshes/robot_parts/wheel2.stl" scale="0.001 0.001 0.001"/>
       </geometry>
       <origin rpy="0 0 0" xyz="0 0 0"/>
@@ -201,6 +201,6 @@
     <origin rpy="0 0 0" xyz="0 -0.1 0"/>
     <axis xyz="0 1 0" />
-    <limit effort="50" velocity="10000"/> <!-- lower="-1.570796327" upper="1.570796327"/> -->
-    <dynamics damping="5" friction="1"/>
+    <limit effort="500" velocity="1000"/> <!-- lower="-1.570796327" upper="1.570796327"/> 6.283-->
+    <dynamics damping="0.01" friction="0.1"/>
   </joint>
   <transmission name="wheel_right_trans">
@@ -334,12 +334,18 @@
 	<gazebo reference="wheel_left_link">
 		<material value="Gazebo/Red"/>
-    <mu1>100.0</mu1>
-    <mu2>100.0</mu2>
+    <mu1>0.7</mu1>
+    <mu2>0.7</mu2>
+    <minDepth>0.001</minDepth>
+    <kp>40000000.0</kp>
+    <kd>0.5</kd>
 	</gazebo>
   <!-- wheel_right_link -->
 	<gazebo reference="wheel_right_link">
 		<material value="Gazebo/Green"/>
-    <mu1>100.0</mu1>
-    <mu2>100.0</mu2>
+    <mu1>0.7</mu1>
+    <mu2>0.7</mu2>
+    <minDepth>0.005</minDepth>
+    <kp>40000000.0</kp>
+    <kd>0.5</kd>
 	</gazebo>
   <gazebo>
